File: kicad/g-1000dxc.kicad_sch (KiCad schematic)
At the start: 53 parts, among them J1001 16V AC, J1005 Screw_Terminal_01x05, J1010 Screw_Terminal_01x07, M01 Indicator Motor (RF-510T-1260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, Q1001 L7805CV-DG, Q1038 L7812CV, U1 Feather, U2 L293D, U3 TLV2372

Commit message: Small bug fix in the schematic
Connections:
- net at U2.1 (EN1,2): now also R12.1; no longer U1.19 (A6/IO14)
- net at R12.2: now also U1.19 (A6/IO14); no longer U1.5 (DAC2/A0)
- net at U2.2 (1A): now also U1.5 (DAC2/A0); no longer R12.1
Changed lines of the file:
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@@
-    (stroke (width 0) (type default) (color 0 0 0 0))
-  )
-  (wire (pts (xy 77.47 82.55) (xy 161.29 82.55))
     (stroke (width 0) (type default) (color 0 0 0 0))
   )
@@
     (stroke (width 0) (type default) (color 0 0 0 0))
   )
-  (wire (pts (xy 157.48 105.41) (xy 163.83 105.41))
-    (stroke (width 0) (type default) (color 0 0 0 0))
-  )
   (wire (pts (xy 77.47 62.23) (xy 77.47 49.53))
     (stroke (width 0) (type default) (color 0 0 0 0))
@@
     (stroke (width 0) (type default) (color 0 0 0 0))
   )
+  (wire (pts (xy 77.47 82.55) (xy 148.59 82.55))
+    (stroke (width 0) (type default) (color 0 0 0 0))
+  )
   (wire (pts (xy 92.71 29.21) (xy 77.47 29.21))
     (stroke (width 0) (type default) (color 0 0 0 0))
@@
     (stroke (width 0) (type default) (color 0 0 0 0))
   )
+  (wire (pts (xy 156.21 82.55) (xy 161.29 82.55))
+    (stroke (width 0) (type default) (color 0 0 0 0))
+  )
   (wire (pts (xy 55.88 90.17) (xy 55.88 92.71))
     (stroke (width 0) (type default) (color 0 0 0 0))
@@
     (stroke (width 0) (type default) (color 0 0 0 0))
   )
-  (wire (pts (xy 111.76 105.41) (xy 149.86 105.41))
+  (wire (pts (xy 111.76 105.41) (xy 163.83 105.41))
     (stroke (width 0) (type default) (color 0 0 0 0))
   )
@@
     )
     (pin "1")
+  )
+  (symbol (lib_id "Device:R") (at 152.4 82.55 270) (unit 1)
+    (in_bom yes) (on_board yes)
+    (property "Reference" "R12" (id 0) (at 151.13 80.01 90)
+      (effects (font (size 1.27 1.27)) (justify right))
+    )
+    (property "Value" "470" (id 1) (at 156.21 80.01 90)
+      (effects (font (size 1.27 1.27)) (justify right))
+    )
+    (property "Footprint" "" (id 2) (at 152.4 80.772 90)
+      (effects (font (size 1.27 1.27)) hide)
+    )
+    (property "Datasheet" "~" (id 3) (at 152.4 82.55 0)
+      (effects (font (size 1.27 1.27)) hide)
+    )
+    (pin "1")
+    (pin "2")
   )
   (symbol (lib_id "Device:R") (at 120.65 175.26 270) (unit 1)
@@
     (pin "2")
   )
-  (symbol (lib_id "Device:R") (at 153.67 105.41 270) (unit 1)
-    (in_bom yes) (on_board yes)
-    (property "Reference" "R12" (id 0) (at 152.4 102.87 90)
-      (effects (font (size 1.27 1.27)) (justify right))
-    )
-    (property "Value" "470" (id 1) (at 157.48 102.87 90)
-      (effects (font (size 1.27 1.27)) (justify right))
-    )
-    (property "Footprint" "" (id 2) (at 153.67 103.632 90)
-      (effects (font (size 1.27 1.27)) hide)
-    )
-    (property "Datasheet" "~" (id 3) (at 153.67 105.41 0)
-      (effects (font (size 1.27 1.27)) hide)
-    )
-    (pin "1")
-    (pin "2")
-  )
   (symbol (lib_id "Device:C") (at 45.72 57.15 90) (unit 1)
     (in_bom yes) (on_board yes)
@@
       (reference "R11") (unit 1) (value "470") (footprint "")
     )
-    (path "/ca8c2319-c7b4-4987-ae25-e9a254752cc0"
+    (path "/297a76ef-3f94-4fbf-b631-f28b81dbe123"
       (reference "R12") (unit 1) (value "470") (footprint "")
     )
